File: proto_E732G4M08S1C/usb_hub.kicad_sch (KiCad schematic)
At the start: 0 parts

Commit message: chg(pcb) more MCU and usb
Parts:
- added U6: FE1.1, Package_QFP:LQFP-48_7x7mm_P0.5mm, symbol PCM_marbastlib-various:FE1.1
Changed lines of the file:
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@@
 	(generator_version "9.0")
 	(paper "A4")
+	(symbol
+		(lib_id "PCM_marbastlib-various:FE1.1")
+		(at 148.59 83.82 0)
+		(unit 1)
+		(exclude_from_sim no)
+		(in_bom yes)
+		(on_board yes)
+		(dnp no)
+		(fields_autoplaced yes)
+		(property "Reference" "U6"
+			(at 159.6233 119.38 0)
+			(effects
+				(font
+					(size 1.27 1.27)
+				)
+				(justify left)
+			)
+		)
+		(property "Value" "FE1.1"
+			(at 159.6233 121.92 0)
+			(effects
+				(font
+					(size 1.27 1.27)
+				)
+				(justify left)
+			)
+		)
+		(property "Footprint" "Package_QFP:LQFP-48_7x7mm_P0.5mm"
+			(at 148.59 69.85 0)
+			(effects
+				(font
+					(size 1.27 1.27)
+				)
+				(hide yes)
+			)
+		)
+		(property "Datasheet" "https://elinux.org/images/e/ee/FE11-datasheet.pdf"
+			(at 148.59 69.85 0)
+			(effects
+				(font
+					(size 1.27 1.27)
+				)
+				(hide yes)
+			)
+		)
+		(property "Description" "4 port USB 2.0 High-Speed (480 Mbit/s) hub with multiple transaction translator"
+			(at 148.59 83.82 0)
+			(effects
+				(font
+					(size 1.27 1.27)
+				)
+				(hide yes)
+			)
+		)
+		(pin "46"
+		)
+		(pin "2"
+		)
+		(pin "44"
+		)
+		(pin "18"
+		)
+		(pin "26"
+		)
+		(pin "13"
+		)
+		(pin "17"
+		)
+		(pin "15"
+		)
+		(pin "42"
+		)
+		(pin "25"
+		)
+		(pin "33"
+		)
+		(pin "39"
+		)
+		(pin "14"
+		)
+		(pin "37"
+		)
+		(pin "5"
+		)
+		(pin "8"
+		)
+		(pin "36"
+		)
+		(pin "30"
+		)
+		(pin "31"
+		)
+		(pin "34"
+		)
+		(pin "11"
+		)
+		(pin "12"
+		)
+		(pin "22"
+		)
+		(pin "20"
+		)
+		(pin "29"
+		)
+		(pin "23"
+		)
+		(pin "1"
+		)
+		(pin "45"
+		)
+		(pin "21"
+		)
+		(pin "3"
+		)
+		(pin "43"
+		)
+		(pin "35"
+		)
+		(pin "48"
+		)
+		(pin "10"
+		)
+		(pin "16"
+		)
+		(pin "40"
+		)
+		(pin "28"
+		)
+		(pin "4"
+		)
+		(pin "9"
+		)
+		(pin "7"
+		)
+		(pin "38"
+		)
+		(pin "24"
+		)
+		(pin "6"
+		)
+		(pin "41"
+		)
+		(pin "47"
+		)
+		(pin "19"
+		)
+		(pin "49"
+		)
+		(pin "27"
+		)
+		(pin "32"
+		)
+		(instances
+			(project ""
+				(path "/3062eac5-ad35-4bd4-9fe0-12754d69cac0/6b08140a-7bb8-4cc8-afd1-e733291ab7cb"
+					(reference "U6")
+					(unit 1)
+				)
+			)
+		)
+	)
 )
