File: proto_E732G4M08S1C/ufp_usb.kicad_sch (KiCad schematic)
At the start: 10 parts, among them J1 USB4510-03-1-A, U1 FUSB302B01MPX, U2 SRV05-4

Commit message: feat(pcb) initial blocks and MCU
Parts:
- C1, C2: footprint Capacitor_SMD:C_1206_3216Metric -> Capacitor_SMD:C_0402_1005Metric
Changed lines of the file:
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@@
 			)
 		)
-		(property "Footprint" "Capacitor_SMD:C_1206_3216Metric"
+		(property "Footprint" "Capacitor_SMD:C_0402_1005Metric"
 			(at 115.2652 76.2 0)
 			(effects
@@
 			)
 		)
-		(property "Footprint" "Capacitor_SMD:C_1206_3216Metric"
+		(property "Footprint" "Capacitor_SMD:C_0402_1005Metric"
 			(at 125.4252 76.2 0)
 			(effects

Commit message: chg(pcb) more MCU and usb
Parts:
- C1, C2: footprint Capacitor_SMD:C_0402_1005Metric -> Capacitor_SMD:C_0603_1608Metric
- R1, R2, R3: footprint Resistor_SMD:R_1206_3216Metric -> Resistor_SMD:R_0603_1608Metric
Changed lines of the file:
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@@
 			)
 		)
-		(property "Footprint" "Resistor_SMD:R_1206_3216Metric"
+		(property "Footprint" "Resistor_SMD:R_0603_1608Metric"
 			(at 68.072 82.55 90)
 			(effects
@@
 			)
 		)
-		(property "Footprint" "Capacitor_SMD:C_0402_1005Metric"
+		(property "Footprint" "Capacitor_SMD:C_0603_1608Metric"
 			(at 115.2652 76.2 0)
 			(effects
@@
 			)
 		)
-		(property "Footprint" "Capacitor_SMD:C_0402_1005Metric"
+		(property "Footprint" "Capacitor_SMD:C_0603_1608Metric"
 			(at 125.4252 76.2 0)
 			(effects
@@
 			)
 		)
-		(property "Footprint" "Resistor_SMD:R_1206_3216Metric"
+		(property "Footprint" "Resistor_SMD:R_0603_1608Metric"
 			(at 83.312 82.55 90)
 			(effects
@@
 			)
 		)
-		(property "Datasheet" "https://gct.co/files/specs/usb4510-spec.pdf"
+		(property "Datasheet" "https://www.usb.org/sites/default/files/documents/usb_type-c.zip"
 			(at 215.9 92.71 0)
 			(effects
@@
 			)
 		)
-		(property "Description" "USB Type C Receptacle for USB 2.0, SMT Type, Mid Mount, 1.6mm Offset"
+		(property "Description" "USB 2.0-only 16P Type-C Receptacle connector"
 			(at 219.71 92.71 0)
 			(effects
@@
 			)
 		)
-		(property "Footprint" "Resistor_SMD:R_1206_3216Metric"
+		(property "Footprint" "Resistor_SMD:R_0603_1608Metric"
 			(at 75.692 82.55 90)
 			(effects

Commit message: feat(pcb) more changes
Connections:
- net CC1: now also U2.4 (IO3)
- net CC2: now also U2.3 (IO2)
- net 3V3 renamed +3.3V
Changed lines of the file:
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@@
+	(wire
+		(pts
+			(xy 144.78 123.19) (xy 147.32 123.19)
+		)
+		(stroke
+			(width 0)
+			(type default)
+		)
+	)
 	(wire
 		(pts
@@
 	(wire
 		(pts
+			(xy 172.72 118.11) (xy 175.26 118.11)
+		)
+		(stroke
+			(width 0)
+			(type default)
+		)
+	)
+	(wire
+		(pts
 			(xy 198.12 74.93) (xy 198.12 77.47)
 		)
@@
 			(width 0)
 			(type default)
+		)
+	)
+	(label "CC2"
+		(at 144.78 123.19 180)
+		(effects
+			(font
+				(size 1.27 1.27)
+			)
+			(justify right bottom)
+		)
+	)
+	(label "CC1"
+		(at 175.26 118.11 0)
+		(effects
+			(font
+				(size 1.27 1.27)
+			)
+			(justify left bottom)
 		)
 	)
@@
 			)
 		)
-		(property "Value" "3V3"
+		(property "Value" "+3.3V"
 			(at 85.09 72.39 0)
 			(effects
@@
 			)
 		)
-		(property "Value" "3V3"
+		(property "Value" "+3.3V"
 			(at 77.47 72.39 0)
 			(effects
@@
 			)
 		)
-		(property "Value" "3V3"
+		(property "Value" "+3.3V"
 			(at 69.85 72.39 0)
 			(effects
